File: DRV8323_BreakoutBoard.kicad_sch (KiCad schematic)
At the start: 36 parts, among them J2 Conn_01x09_Pin, J4 Conn_01x02_Pin, J6 Conn_01x09_Pin, Q1 30v_60a_Mosfet, Q2 30v_60a_Mosfet, Q3 30v_60a_Mosfet, Q4 30v_60a_Mosfet, Q5 30v_60a_Mosfet, Q6 30v_60a_Mosfet, U6 DRV8323S

Commit message: V0
Parts:
- removed C20, C24, C26: C_0603_1uF, Capacitor_SMD:C_0603_1608Metric, symbol PCM_Capacitor_AKL:C_0805
- added C2, C4, C5: C_0805_10uF, Capacitor_SMD:C_0805_2012Metric, symbol PCM_Capacitor_AKL:C_0805
- added C3: Cap_D12.5mm_1000uF, PCM_Capacitor_THT_AKL:CP_Radial_D12.5mm_P5.00mm, symbol PCM_Capacitor_AKL:CP_Radial_D12.5mm_P5.00mm
Connections:
- net GND: now also C2.1, C3.2, C4.1, C5.1
- net SOA: now also J6.3 (Pin_3); no longer J6.1 (Pin_1)
- net SOC: now also J6.1 (Pin_1); no longer J6.3 (Pin_3)
- net VIN: now also C2.2, C3.1, C4.2, C5.2
Other:
- moved on the sheet: J4
